Commit message: feat(crx): load calibrated wrist camera and TCP from calibration store
- add crx_calibration_args.xacro (wrist_camera, camera_calibration, tcp_calibration) included by crx10ia*.xacro
- resolve active ~/.ros/calibration current.yaml in robot_bringup.launch.py, falling back to crx_description defaults
- add default calibration YAMLs (Femto, D435, welding TCP) and crx10ia_l_cell / wrist camera xacros
- update MoveIt srdf, joint_limits, ompl and kinematics for the CRX models
- add tools/fake_fanuc_controller.py for testing without a robot

Co-Authored-By: Claude Opus 5.5 <noreply@anthropic.com>

File: crx_description/urdf/crx10ia/crx10ia.urdf.xacro (robot description, xacro)
@@ -6,5 +6,7 @@
               use_rmi:='false'
               use_mock_hardware:=false
-              gz:=false">
+              gz:=false
+              tcp_xyz:='0 0 0'
+              tcp_rpy:='0 ${pi/2} 0'">
     <xacro:if value="${gz}">
       <xacro:include filename="$(find crx_description)/urdf/crx.gazebo.xacro" />
@@ -190,6 +192,7 @@
     <!-- tcp -->
     <link name="tcp" />
+    <!-- tcp_xyz/tcp_rpy: welding TCP from the calibration store (top-level crx10ia*.xacro). -->
     <joint name="flange-tcp" type="fixed">
-      <origin xyz="0 0 0" rpy="0 ${pi/2} 0" />
+      <origin xyz="${tcp_xyz}" rpy="${tcp_rpy}" />
       <parent link="flange" />
       <child link="tcp" />

File: crx_description/urdf/crx10ia/crx10ia.xacro (robot description, xacro)
@@ -6,4 +6,6 @@
   <xacro:arg name="use_rmi" default="false" />
   <xacro:include filename="$(find crx_description)/urdf/crx10ia/crx10ia.urdf.xacro"/>
-  <xacro:crx10ia use_mock_hardware="$(arg use_mock_hardware)" robot_ip="$(arg robot_ip)" read_only="$(arg read_only)" use_rmi="$(arg use_rmi)"/>
+  <xacro:include filename="$(find crx_description)/urdf/include/crx_calibration_args.xacro"/>
+  <xacro:crx10ia use_mock_hardware="$(arg use_mock_hardware)" robot_ip="$(arg robot_ip)" read_only="$(arg read_only)" use_rmi="$(arg use_rmi)" tcp_xyz="${crx_tcp_origin['xyz']}" tcp_rpy="${crx_tcp_origin['rpy']}"/>
+  <xacro:crx_calibrated_wrist_camera/>
 </robot>

File: crx_description/urdf/crx10ia_l/crx10ia_l.urdf.xacro (robot description, xacro)
@@ -6,5 +6,7 @@
               use_rmi:='false'
               use_mock_hardware:=false
-              gz:=false">
+              gz:=false
+              tcp_xyz:='0 0 0'
+              tcp_rpy:='0 ${pi/2} 0'">
     <xacro:if value="${gz}">
       <xacro:include filename="$(find crx_description)/urdf/crx.gazebo.xacro" />
@@ -190,6 +192,7 @@
     <!-- tcp -->
     <link name="tcp" />
+    <!-- tcp_xyz/tcp_rpy: welding TCP from the calibration store (top-level crx10ia*.xacro). -->
     <joint name="flange-tcp" type="fixed">
-      <origin xyz="0 0 0" rpy="0 ${pi/2} 0" />
+      <origin xyz="${tcp_xyz}" rpy="${tcp_rpy}" />
       <parent link="flange" />
       <child link="tcp" />

File: crx_description/urdf/crx10ia_l/crx10ia_l.xacro (robot description, xacro)
@@ -6,5 +6,13 @@
   <xacro:arg name="use_rmi" default="false" />
   <xacro:arg name="gz" default="false" />
+  <!-- welding cell digital twin (table, pedestal, positioner), see crx10ia_l_cell.xacro -->
+  <xacro:arg name="cell" default="true" />
   <xacro:include filename="$(find crx_description)/urdf/crx10ia_l/crx10ia_l.urdf.xacro"/>
-  <xacro:crx10ia_l use_mock_hardware="$(arg use_mock_hardware)" robot_ip="$(arg robot_ip)" read_only="$(arg read_only)" use_rmi="$(arg use_rmi)" gz="$(arg gz)" />
+  <xacro:include filename="$(find crx_description)/urdf/include/crx_calibration_args.xacro"/>
+  <xacro:crx10ia_l use_mock_hardware="$(arg use_mock_hardware)" robot_ip="$(arg robot_ip)" read_only="$(arg read_only)" use_rmi="$(arg use_rmi)" gz="$(arg gz)" tcp_xyz="${crx_tcp_origin['xyz']}" tcp_rpy="${crx_tcp_origin['rpy']}"/>
+  <xacro:crx_calibrated_wrist_camera/>
+  <xacro:if value="$(arg cell)">
+    <xacro:include filename="$(find crx_description)/urdf/crx10ia_l/crx10ia_l_cell.xacro"/>
+    <xacro:crx10ia_l_cell parent="base_link"/>
+  </xacro:if>
 </robot>
