Commit message: feat(crx_description): primitive welding-torch collision from the active TCP
crx_torch_collision.xacro builds torch_neck (parallel to the flange axis
through the neck bend, so an off-centre bracket needs no measured offset),
torch_nozzle (on the wire axis) and torch_wire (stick-out, visual only by
default) on `flange` from the TCP calibration. Dimensions come from
config/torch_collision.yaml, overridden by the TCP version's `torch` block
(GUI Apply). Nothing is generated for an uncalibrated TCP. The CRX-10iA(/L)
SRDFs disable the torch only against link_6 and the wrist camera.

Co-Authored-By: Claude Opus 5.5 <noreply@anthropic.com>

File: crx_description/urdf/crx10ia/crx10ia.xacro (robot description, xacro)
@@ -9,3 +9,4 @@
   <xacro:crx10ia use_mock_hardware="$(arg use_mock_hardware)" robot_ip="$(arg robot_ip)" read_only="$(arg read_only)" use_rmi="$(arg use_rmi)" tcp_xyz="${crx_tcp_origin['xyz']}" tcp_rpy="${crx_tcp_origin['rpy']}"/>
   <xacro:crx_calibrated_wrist_camera/>
+  <xacro:crx_calibrated_torch_collision/>
 </robot>

File: crx_description/urdf/crx10ia_l/crx10ia_l.xacro (robot description, xacro)
@@ -12,4 +12,5 @@
   <xacro:crx10ia_l use_mock_hardware="$(arg use_mock_hardware)" robot_ip="$(arg robot_ip)" read_only="$(arg read_only)" use_rmi="$(arg use_rmi)" gz="$(arg gz)" tcp_xyz="${crx_tcp_origin['xyz']}" tcp_rpy="${crx_tcp_origin['rpy']}"/>
   <xacro:crx_calibrated_wrist_camera/>
+  <xacro:crx_calibrated_torch_collision/>
   <xacro:if value="$(arg cell)">
     <xacro:include filename="$(find crx_description)/urdf/crx10ia_l/crx10ia_l_cell.xacro"/>

File: crx_description/urdf/include/crx_calibration_args.xacro (robot description, xacro)
@@ -6,4 +6,5 @@
     camera_calibration  mount YAML ('' = crx_description default for wrist_camera)
     tcp_calibration     TCP YAML, its `real` origin is flange -> tcp ('' = crx_description default)
+    torch_collision     torch collision dimensions YAML ('' = crx_description config/torch_collision.yaml)
   GUI launches pass the robot's active ~/.ros/calibration/<robot_id>/... current.yaml
   (hand_eye_calibration/calibration_store.py), so Apply = new version + push.
@@ -13,6 +14,8 @@
   <xacro:arg name="camera_calibration" default=""/>
   <xacro:arg name="tcp_calibration" default=""/>
+  <xacro:arg name="torch_collision" default=""/>
   <xacro:property name="crx_wrist_camera" value="$(arg wrist_camera)"/>
-  <xacro:property name="crx_tcp_origin" value="${xacro.load_yaml('$(arg tcp_calibration)' or '$(find crx_description)/config/calibration/welding_tcp_default.yaml')['real']}"/>
+  <xacro:property name="crx_tcp_yaml" value="${xacro.load_yaml('$(arg tcp_calibration)' or '$(find crx_description)/config/calibration/welding_tcp_default.yaml')}"/>
+  <xacro:property name="crx_tcp_origin" value="${crx_tcp_yaml['real']}"/>
   <xacro:macro name="crx_calibrated_wrist_camera">
     <xacro:if value="${crx_wrist_camera in ('femto_bolt', 'realsense_d435')}">
@@ -22,3 +25,11 @@
     </xacro:if>
   </xacro:macro>
+  <!-- Primitive welding-torch collision built from the active TCP (crx_torch_collision.xacro).
+       Dimensions: torch_collision YAML, overridden by the TCP version's `torch` block (GUI Apply). -->
+  <xacro:macro name="crx_calibrated_torch_collision">
+    <xacro:include filename="$(find crx_description)/urdf/include/crx_torch_collision.xacro"/>
+    <xacro:property name="torch_defaults" value="${xacro.load_yaml('$(arg torch_collision)' or '$(find crx_description)/config/torch_collision.yaml')}"/>
+    <xacro:crx_torch_collision tcp="${crx_tcp_origin}"
+      cfg="${dict(list(torch_defaults.items()) + list((crx_tcp_yaml.get('torch') or dict()).items()))}"/>
+  </xacro:macro>
 </robot>
